File: KiCAD/K65-SBC.sch (KiCad schematic (older format))
At the start: 24 parts, among them J1 SERIAL CON, SW1 RESET, U1 74HC04, U2 W65C02SxP, U3 74HC74, U4 74HC00, U5 MC6850, U6 28C256, U7 62256, Y1 7.3728MHz

Commit message: 回路図整備、部品表作成
Parts:
- added C1, C2, C3, C4: 0.1u, symbol Device:C_Small
- added C11: 10u, symbol Device:CP
- added D2: POWER LED, symbol Device:LED_ALT
- added J3: DC JACK, symbol Connector:Barrel_Jack_Switch
- added R4: 470, symbol Device:R_US
- added SW2: POWER SW, symbol Switch:SW_SPST
- R3: value R_US -> 1k
- gave numbers to parts that had none: 2
- renumbered C6 to C10, C2 to C5, C1 to C6, C3 to C7, C4 to C8, C5 to C9, RN1 to RN3, U6 to U1, U7 to U2, U5 to U3, U2 to U4, U4 to U5, U3 to U6, U1 to U7
Connections:
- net labels removed: E, RESET
- wire segments 313 -> 345

Commit message: REV1ガーバーデータ出力
Parts:
- added H1, H2, H3, H4: MountingHole, MountingHole:MountingHole_3.2mm_M3, symbol Mechanical:MountingHole
- C1, C10, C2, C3, C4, C6, C7, C8, C9: footprint (none) -> Capacitor_THT:C_Disc_D3.0mm_W1.6mm_P2.50mm
- C11, C5: footprint (none) -> Capacitor_THT:CP_Radial_D5.0mm_P2.50mm
- D1: footprint (none) -> Diode_THT:D_DO-34_SOD68_P10.16mm_Horizontal
- D2: footprint (none) -> LED_THT:LED_D3.0mm
- J1: footprint (none) -> Connector_PinHeader_2.54mm:PinHeader_1x06_P2.54mm_Horizontal
- J2: footprint (none) -> Connector_PinHeader_2.54mm:PinHeader_2x20_P2.54mm_Horizontal
- J3: footprint (none) -> Connector_BarrelJack:BarrelJack_Horizontal
- R1, R2, R3, R4: footprint (none) -> Resistor_THT:R_Axial_DIN0207_L6.3mm_D2.5mm_P10.16mm_Horizontal
- SW1: footprint (none) -> Button_Switch_THT:SW_PUSH_6mm
- SW2: footprint (none) -> Connector_PinHeader_2.54mm:PinHeader_1x03_P2.54mm_Vertical
- U1: footprint (none) -> Package_TO_SOT_THT:TO-92_Inline_Wide
- U2: footprint (none) -> Package_DIP:DIP-28_W15.24mm_Socket_LongPads
- U3: footprint Package_DIP:DIP-40_W15.24mm -> Package_DIP:DIP-24_W15.24mm_Socket_LongPads
- U4: footprint (none) -> Package_DIP:DIP-40_W15.24mm_Socket_LongPads; symbol 65xx:W65C02SxP -> K65-SBC-rescue:W65C02SxP-65xx
- U5, U6, U7: footprint (none) -> Package_DIP:DIP-14_W7.62mm_Socket_LongPads
- Y1: footprint (none) -> Crystal:Crystal_HC50_Vertical
